Commit message: Added humanoid to gazebo

File: description/humanoid_core.xacro (robot description, xacro)
@@ -52,4 +52,7 @@
         </collision>
     </link>
+    <gazebo reference="base_link">
+        <material>Gazebo/Blue</material>
+    </gazebo>
     <link
         name="Right_leg">
@@ -150,4 +153,7 @@
         </collision>
     </link>
+    <gazebo reference="rl1">
+        <material>Gazebo/Black</material>
+    </gazebo>
     <joint
         name="rlj1"
@@ -266,4 +272,7 @@
         </collision>
     </link>
+    <gazebo reference="rl3">
+        <material>Gazebo/Black</material>
+    </gazebo>
     <joint
         name="rlj3"
@@ -382,4 +391,7 @@
         </collision>
     </link>
+    <gazebo reference="rl5">
+        <material>Gazebo/Black</material>
+    </gazebo>
     <joint
         name="rlj5"
@@ -498,4 +510,7 @@
         </collision>
     </link>
+    <gazebo reference="ll1">
+        <material>Gazebo/Black</material>
+    </gazebo>
     <joint
         name="llj1"
@@ -614,4 +629,7 @@
         </collision>
     </link>
+    <gazebo reference="ll3">
+        <material>Gazebo/Black</material>
+    </gazebo>
     <joint
         name="llj3"
@@ -730,4 +748,7 @@
         </collision>
     </link>
+    <gazebo reference="ll5">
+        <material>Gazebo/Black</material>
+    </gazebo>
     <joint
         name="llj5"
@@ -846,4 +867,7 @@
         </collision>
     </link>
+    <gazebo reference="rh1">
+        <material>Gazebo/Black</material>
+    </gazebo>
     <joint
         name="rhj1"
@@ -962,4 +986,7 @@
         </collision>
     </link>
+    <gazebo reference="rh3">
+        <material>Gazebo/Black</material>
+    </gazebo>
     <joint
         name="rhj3"
@@ -1078,4 +1105,7 @@
         </collision>
     </link>
+    <gazebo reference="lh1">
+        <material>Gazebo/Black</material>
+    </gazebo>
     <joint
         name="lhj1"
@@ -1194,4 +1224,7 @@
         </collision>
     </link>
+    <gazebo reference="lh3">
+        <material>Gazebo/Black</material>
+    </gazebo>
     <joint
         name="lhj3"
